Commit message: organize the files deleted

File: Rviz_AngleDisplay_test/src/robot_description/urdf/rr_position_control.urdf (robot description, URDF)
Before this commit: robot rr_position_control, 3 links, 2 joints
Joints:
- joint RR_position_control_joint2: origin xyz=0 0 0.1 rpy=0 0 0 -> xyz=0 0 0.2 rpy=0 0 0
